Commit message: fixing time problems

File: simulation/xacro/Doris.xacro (robot description, xacro)
@@ -4,5 +4,5 @@
 		<inertial>
 			<inertia  ixx="1.0" ixy="0.0"  ixz="0.0"  iyy="1.0"  iyz="0.0"  izz="1.0" />	                <origin xyz = "0 0 0.165" rpy ="0 0 0"/>
-			<mass value= "10" />
+			<mass value= "50" />
 		</inertial>
 		<visual>

File: simulation/xacro/mycasterwheel.xacro (robot description, xacro)
@@ -11,31 +11,25 @@
 			<mass value = "0.5"/>
 			<origin xyz="0 0 0" rpy="0 0 0"/>
-			<inertia ixx="1" ixy="0" ixz="0" iyy="1" iyz="0" izz="1" />
+			 <inertia ixx="0.001" ixy="0.0" ixz="0.0" iyy="0.001" iyz="0.0" izz="0.001"/>
 		</inertial>
-	<collision>
-		<origin xyz="0 0 0" rpy="0 0 0"/>
-		<geometry>
-			<sphere radius="0.05"/>
-		</geometry>
-		<gazebo>
-			<surface>
-			  <friction>
-			    <ode>
-			      <mu>0</mu>
-			      <mu2>0</mu2>
-			      <slip1>1.0</slip1>
-			      <slip2>1.0</slip2>
-			    </ode>
-			  </friction>
-			</surface>
-		</gazebo>
-	</collision>
-	<visual>
-		<origin xyz="0 0 0" rpy="0 0 0"/>
-		<geometry>
-			<sphere radius="0.05"/>
-		</geometry>
-	</visual>
+		<collision>
+			<origin xyz="0 0 0" rpy="0 0 0"/>
+			<geometry>
+				<sphere radius="0.05"/>
+			</geometry>
+		</collision>
+		<visual>
+			<origin xyz="0 0 0" rpy="0 0 0"/>
+			<geometry>
+				<sphere radius="0.05"/>
+			</geometry>
+		</visual>
 	</link>
+	<gazebo reference ="${prefix}_link">
+		<mu1 value="0.0"/>
+    		<mu2 value="0.0"/>
+    		<kp value="10000000.0"/>
+    		<kd value="0.00001"/>
+	</gazebo>
 </xacro:macro>
 </robot>

Commit message: navigation_files

File: simulation/xacro/Doris.xacro (robot description, xacro)
@@ -4,5 +4,5 @@
 		<inertial>
 			<inertia  ixx="1.0" ixy="0.0"  ixz="0.0"  iyy="1.0"  iyz="0.0"  izz="1.0" />	                <origin xyz = "0 0 0.165" rpy ="0 0 0"/>
-			<mass value= "50" />
+			<mass value= "80" />
 		</inertial>
 		<visual>

Commit message: fixing amcl and new world

File: simulation/xacro/Doris.xacro (robot description, xacro)
@@ -19,10 +19,10 @@
 		</collision>
 	</link>
-	<joint name="right_axis" type="revolute" >
+	<joint name="right_axis" type="continuous" >
 		<origin xyz = "0 -0.15 0" rpy ="0 0 0"/>
 		<parent link = "cuerpo"/>
 		<child link= "right_wheel"/>
 		<axis xyz="0 1 0"/>
-		<limit effort="30" velocity="0.1" lower="${-2*pi}" upper="${2*pi}"/>
+		<!--<limit effort="30" velocity="0.1" lower="${-2*pi}" upper="${2*pi}"/>-->
 	</joint>
 	<link name='right_wheel'>
@@ -44,10 +44,10 @@
 		</collision>
 	</link>
-	<joint name="left_axis" type="revolute" >
+	<joint name="left_axis" type="continuous" >
 		<origin xyz = "0 0.15 0" rpy ="0 0 0"/>
 		<parent link = "cuerpo"/>
 		<child link= "left_wheel"/>
 		<axis xyz="0 1 0"/>
-		<limit effort="30" velocity="0.1" lower="${-2*pi}" upper="${2*pi}"/>
+		<!--<limit effort="30" velocity="0.1" lower="${-2*pi}" upper="${2*pi}"/>-->
 	</joint>
 	<link name='left_wheel'>

File: simulation/xacro/mycasterwheel.xacro (robot description, xacro)
@@ -9,5 +9,5 @@
 	<link name="${prefix}_link">
 		<inertial>
-			<mass value = "0.5"/>
+			<mass value = "0.1"/>
 			<origin xyz="0 0 0" rpy="0 0 0"/>
 			 <inertia ixx="0.001" ixy="0.0" ixz="0.0" iyy="0.001" iyz="0.0" izz="0.001"/>
